Commit message: updated gym bridge code for rviz and added requirements.txt

File: src/simulator/launch/ego_racecar.xacro (robot description, xacro)
@@ -5,4 +5,5 @@
   <xacro:property name="width" value="0.2032" />
   <xacro:property name="height" value="0.1" />
+  <!-- <xacro:property name="pi" value="3.14159265359"/> -->
   <xacro:property name="ground_offset" value="0.04" />
   <xacro:property name="wheel_radius" value="0.0508" />
